Commit message: 1

File: assets/roboparty_atom01_long/atom01_long.urdf (robot description, URDF)
Before this commit: robot atom01urdf, 24 links, 23 joints
Links:
- link base_link: mass 5.38006123 -> 5.46006
- link left_ankle_pitch_link: mass 0.084 -> 0.08400
- link left_ankle_roll_link: mass 0.30640039  -> 0.20002
- link left_knee_link: mass 1.79036871 -> 1.73050; geometry collision box name=left_knee_link size=0.08 0.08 0.22; visual mesh filename=./meshes/left_knee_link.STL
- link left_thigh_pitch_link: mass 2.34600762 -> 2.31922
- link left_thigh_roll_link: mass 1.71632646 -> 1.67349
- link left_thigh_yaw_link: mass 1.68866185 -> 1.67364
- link right_ankle_pitch_link: mass 0.084 -> 0.08400
- link right_ankle_roll_link: mass  0.30640039 -> 0.20002
- link right_knee_link: mass 1.79036871 -> 1.74926
- link right_thigh_pitch_link: mass 2.34600762 -> 2.31922
- link right_thigh_roll_link: mass 1.71632646 -> 1.67349
- link right_thigh_yaw_link: mass 1.68565743 -> 1.67349
Joints:
- joint left_ankle_pitch_joint: origin xyz=0 -0.02085 -0.3 rpy=0 0 0 -> xyz=0.0199999999548295 -0.0193500000002206 -0.300000000002996 rpy=0 0 0
- joint left_knee_joint: origin xyz=0 0 -0.25 rpy=0 0 0 -> xyz=-5.71909387963032E-05 0 -0.249999999984666 rpy=0 0 0
- joint left_thigh_pitch_joint: origin xyz=0.060622 0.02085 -0.035 rpy=0 0 0 -> xyz=0.0623538151339522 0.0193500079963393 -0.0360000241422042 rpy=0 0 0
- joint left_thigh_roll_joint: origin xyz=-0.017693 0 -0.072346 rpy=0 0 0 -> xyz=-0.019425 0 -0.071346 rpy=0 0 0
- joint left_thigh_yaw_joint: origin xyz=-0.071093 0.0725 -0.051778 rpy=0 0 0 -> xyz=-0.070843 0.10009 -0.051345 rpy=0 0 0
- joint right_ankle_pitch_joint: origin xyz=0 0.0208500000000073 -0.299999999999986 rpy=0 0 0 -> xyz=0.019999999955032 0.0193499999997858 -0.300000000003003 rpy=0 0 0
- joint right_knee_joint: origin xyz=0 0 -0.250000000000016 rpy=0 0 0 -> xyz=0 0 -0.249999999984727 rpy=0 0 0
- joint right_thigh_pitch_joint: origin xyz=0.0619208163652291 -0.0208499999999942 -0.0357500000093095 rpy=0 0 0 -> xyz=0.0619208163651855 -0.0193500000000049 -0.0357500000093318 rpy=0 0 0
- joint right_thigh_roll_joint: axis 0.86603 0 -0.5 -> 0.866025403709328 0 -0.500000000130096; origin xyz=-0.0189924084475403 0 -0.0715958163677252 rpy=0 0 0 -> xyz=-0.018742408447476 0 -0.0711628036658393 rpy=0 0 0
- joint right_thigh_yaw_joint: origin xyz=-0.071093 -0.0725 -0.051778 rpy=0 0 0 -> xyz=-0.071093 -0.099911 -0.051778 rpy=0 0 0

File: assets/roboparty_atom02/atom02.urdf (robot description, URDF)
Before this commit: robot ATOM02, 24 links, 24 joints
Links:
- added link torso_roll_link, mass 1.50165300; collision mesh filename=./meshes/torso_roll_link.STL; visual mesh filename=./meshes/torso_roll_link.STL
- link base_link: mass 0.726960641971639 -> 3.23595958; geometry collision mesh filename=./meshes/base_link.STL; visual mesh filename=./meshes/base_link.STL
- link left_ankle_pitch_link: mass 0.177201152706737 -> 0.22519575; geometry collision mesh filename=./meshes/left_ankle_pitch_link.STL; visual mesh filename=./meshes/left_ankle_pitch_link.STL
- link left_ankle_roll_link: mass 1.3391 -> 0.58290878; geometry collision mesh filename=./meshes/left_ankle_roll_link.STL; visual mesh filename=./meshes/left_ankle_roll_link.STL
- link left_elbow_pitch_link: mass 0.361375425050572 -> 0.88600228; geometry collision mesh filename=./meshes/left_elbow_pitch_link.STL; visual mesh filename=./meshes/left_elbow_pitch_link.STL
- link left_elbow_yaw_link: mass 1.41761671859828 -> 0.23249655; geometry collision mesh filename=./meshes/left_elbow_yaw_link.STL; visual mesh filename=./meshes/left_elbow_yaw_link.STL
- link left_knee_link: mass 27.435138431354 -> 2.18421456; geometry collision mesh filename=./meshes/left_knee_link.STL; visual mesh filename=./meshes/left_knee_link.STL
- link left_shoulder_pitch_link: mass 0.281602434591795 -> 0.68492195; geometry collision mesh filename=./meshes/left_shoulder_pitch_link.STL; visual mesh filename=./meshes/left_shoulder_pitch_link.STL
- link left_shoulder_roll_link: mass 0.294057859644599 -> 0.69553781; geometry collision mesh filename=./meshes/left_shoulder_roll_link.STL; visual mesh filename=./meshes/left_shoulder_roll_link.STL
- link left_shoulder_yaw_link: mass 0.570014294886847 -> 1.01870173; geometry collision mesh filename=./meshes/left_shoulder_yaw_link.STL; visual mesh filename=./meshes/left_shoulder_yaw_link.STL
- link left_thigh_pitch_link: mass 0.556662079227767 -> 1.45950912; geometry collision mesh filename=./meshes/left_thigh_pitch_link.STL; visual mesh filename=./meshes/left_thigh_pitch_link.STL
- link left_thigh_roll_link: mass 2.90711030732957 -> 1.90711030732957; geometry collision mesh filename=./meshes/left_thigh_roll_link.STL; visual mesh filename=./meshes/left_thigh_roll_link.STL
- link left_thigh_yaw_link: mass 25.7162947988607 -> 2.32668441; geometry collision mesh filename=./meshes/left_thigh_yaw_link.STL; visual mesh filename=./meshes/left_thigh_yaw_link.STL
- link right_ankle_pitch_link: mass 0.177201152706736 -> 0.22519575; geometry collision mesh filename=./meshes/right_ankle_pitch_link.STL; visual mesh filename=./meshes/right_ankle_pitch_link.STL
- link right_ankle_roll_link: mass 1.33912671571889 -> 0.58290878; geometry collision mesh filename=./meshes/right_ankle_roll_link.STL; visual mesh filename=./meshes/right_ankle_roll_link.STL
- link right_elbow_pitch_link: mass 0.361375020829954 -> 0.88408116; geometry collision mesh filename=./meshes/right_elbow_pitch_link.STL; visual mesh filename=./meshes/right_elbow_pitch_link.STL
- link right_elbow_yaw_link: mass 1.41764942980355 -> 0.23249633; geometry collision mesh filename=./meshes/right_elbow_yaw_link.STL; visual mesh filename=./meshes/right_elbow_yaw_link.STL
- link right_knee_link: mass 27.4495729659464 -> 2.16342478; geometry collision mesh filename=./meshes/right_knee_link.STL; visual mesh filename=./meshes/right_knee_link.STL
- link right_shoulder_pitch_link: mass 0.281602420918166 -> 0.68494995; geometry collision mesh filename=./meshes/right_shoulder_pitch_link.STL; visual mesh filename=./meshes/right_shoulder_pitch_link.STL
- link right_shoulder_roll_link: mass 0.294057899511326 -> 0.70646494; geometry collision mesh filename=./meshes/right_shoulder_roll_link.STL; visual mesh filename=./meshes/right_shoulder_roll_link.STL
- link right_shoulder_yaw_link: mass 0.570014294602155 -> 1.02101321; geometry collision mesh filename=./meshes/right_shoulder_yaw_link.STL; visual mesh filename=./meshes/right_shoulder_yaw_link.STL
- link right_thigh_pitch_link: mass 0.556662079541713 -> 1.44712395; geometry collision mesh filename=./meshes/right_thigh_pitch_link.STL; visual mesh filename=./meshes/right_thigh_pitch_link.STL
- link right_thigh_roll_link: mass 2.90779917980452 -> 1.91914876; geometry collision mesh filename=./meshes/right_thigh_roll_link.STL; visual mesh filename=./meshes/right_thigh_roll_link.STL
- link right_thigh_yaw_link: mass 24.4949645811454 -> 2.32668364; geometry collision mesh filename=./meshes/right_thigh_yaw_link.STL; visual mesh filename=./meshes/right_thigh_yaw_link.STL
- link torso_yaw_link: mass 0.905363139813927 -> 6.55523381; geometry collision mesh filename=./meshes/torso_yaw_link.STL; visual mesh filename=./meshes/torso_yaw_link.STL
Joints:
- removed joint left_elbow_yaw_link
- removed joint right_shoulder_yaw_link
- added joint left_elbow_yaw_joint: type revolute, parent left_elbow_pitch_link, child left_elbow_yaw_link, origin xyz=0 0 -0.0133504827638016 rpy=0 0 0, axis 1 0 0, limit lower=-3.14159 upper=3.14159 effort=30 velocity=12
- added joint right_shoulder_yaw_joint: type revolute, parent right_shoulder_roll_link, child right_shoulder_yaw_link, origin xyz=0 -0.00647168056291525 0.000825647150946768 rpy=0 0 0, axis 0 0 -1, limit lower=-3.14159 upper=3.14159 effort=30 velocity=12
- joint left_thigh_roll_joint: limit lower=-0.5236 upper=2.6164 effort=140 velocity=12 -> lower=-0.1745 upper=2.6878 effort=140 velocity=12
- joint right_thigh_roll_joint: limit lower=-2.6164 upper=0.5236 effort=140 velocity=12 -> lower=-2.6878 upper=0.1745 effort=140 velocity=12

File: assets/roboparty_atom02/urdf/atom02.urdf (robot description, URDF)
Before this commit: robot ATOM02, 25 links, 24 joints
Links:
- removed link right _thigh_pitch_link
- added link right_thigh_pitch_link, mass 1.44712395; collision mesh filename=../meshes/right_thigh_pitch_link.STL; visual mesh filename=../meshes/right_thigh_pitch_link.STL
- link base_link: mass 0.726960641971639 -> 3.23595958; geometry collision mesh filename=../meshes/base_link.STL; visual mesh filename=../meshes/base_link.STL
- link left_ankle_pitch_link: mass 0.177201152706737 -> 0.22519575; geometry collision mesh filename=../meshes/left_ankle_pitch_link.STL; visual mesh filename=../meshes/left_ankle_pitch_link.STL
- link left_ankle_roll_link: mass 1.3391 -> 0.58290878; geometry collision mesh filename=../meshes/left_ankle_roll_link.STL; visual mesh filename=../meshes/left_ankle_roll_link.STL
- link left_elbow_pitch_link: mass 0.361375425050572 -> 0.88600228; geometry collision mesh filename=../meshes/left_elbow_pitch_link.STL; visual mesh filename=../meshes/left_elbow_pitch_link.STL
- link left_elbow_yaw_link: mass 1.41761671859828 -> 0.23249655; geometry collision mesh filename=../meshes/left_elbow_yaw_link.STL; visual mesh filename=../meshes/left_elbow_yaw_link.STL
- link left_knee_link: mass 27.435138431354 -> 2.18421456; geometry collision mesh filename=../meshes/left_knee_link.STL; visual mesh filename=../meshes/left_knee_link.STL
- link left_shoulder_pitch_link: mass 0.281602434591795 -> 0.68492195; geometry collision mesh filename=../meshes/left_shoulder_pitch_link.STL; visual mesh filename=../meshes/left_shoulder_pitch_link.STL
- link left_shoulder_roll_link: mass 0.294057859644599 -> 0.69553781; geometry collision mesh filename=../meshes/left_shoulder_roll_link.STL; visual mesh filename=../meshes/left_shoulder_roll_link.STL
- link left_shoulder_yaw_link: mass 0.570014294886847 -> 1.01870173; geometry collision mesh filename=../meshes/left_shoulder_yaw_link.STL; visual mesh filename=../meshes/left_shoulder_yaw_link.STL
- link left_thigh_pitch_link: mass 0.556662079227767 -> 1.45950912; geometry collision mesh filename=../meshes/left_thigh_pitch_link.STL; visual mesh filename=../meshes/left_thigh_pitch_link.STL
- link left_thigh_roll_link: mass 2.90711030732957 -> 1.90711030732957; geometry collision mesh filename=../meshes/left_thigh_roll_link.STL; visual mesh filename=../meshes/left_thigh_roll_link.STL
- link left_thigh_yaw_link: mass 25.7162947988607 -> 2.32668441; geometry collision mesh filename=../meshes/left_thigh_yaw_link.STL; visual mesh filename=../meshes/left_thigh_yaw_link.STL
- link right_ankle_pitch_link: mass 0.177201152706736 -> 0.22519575; geometry collision mesh filename=../meshes/right_ankle_pitch_link.STL; visual mesh filename=../meshes/right_ankle_pitch_link.STL
- link right_ankle_roll_link: mass 1.33912671571889 -> 0.58290878; geometry collision mesh filename=../meshes/right_ankle_roll_link.STL; visual mesh filename=../meshes/right_ankle_roll_link.STL
- link right_elbow_pitch_link: mass 0.361375020829954 -> 0.88408116; geometry collision mesh filename=../meshes/right_elbow_pitch_link.STL; visual mesh filename=../meshes/right_elbow_pitch_link.STL
- link right_elbow_yaw_link: mass 1.41764942980355 -> 0.23249633; geometry collision mesh filename=../meshes/right_elbow_yaw_link.STL; visual mesh filename=../meshes/right_elbow_yaw_link.STL
- link right_knee_link: mass 27.4495729659464 -> 2.16342478; geometry collision mesh filename=../meshes/right_knee_link.STL; visual mesh filename=../meshes/right_knee_link.STL
- link right_shoulder_pitch_link: mass 0.281602420918166 -> 0.68494995; geometry collision mesh filename=../meshes/right_shoulder_pitch_link.STL; visual mesh filename=../meshes/right_shoulder_pitch_link.STL
- link right_shoulder_roll_link: mass 0.294057899511326 -> 0.70646494; geometry collision mesh filename=../meshes/right_shoulder_roll_link.STL; visual mesh filename=../meshes/right_shoulder_roll_link.STL
- link right_shoulder_yaw_link: mass 0.570014294602155 -> 1.02101321; geometry collision mesh filename=../meshes/right_shoulder_yaw_link.STL; visual mesh filename=../meshes/right_shoulder_yaw_link.STL
- link right_thigh_roll_link: mass 2.90779917980452 -> 1.91914876; geometry collision mesh filename=../meshes/right_thigh_roll_link.STL; visual mesh filename=../meshes/right_thigh_roll_link.STL
- link right_thigh_yaw_link: mass 24.4949645811454 -> 2.32668364; geometry collision mesh filename=../meshes/right_thigh_yaw_link.STL; visual mesh filename=../meshes/right_thigh_yaw_link.STL
- link torso_roll_link: mass 0 -> 1.50165300; geometry collision mesh filename=../meshes/torso_roll_link.STL; visual mesh filename=../meshes/torso_roll_link.STL
- link torso_yaw_link: mass 0.905363139813927 -> 6.55523381; geometry collision mesh filename=../meshes/torso_yaw_link.STL; visual mesh filename=../meshes/torso_yaw_link.STL
Joints:
- removed joint left_elbow_yaw_link
- removed joint right _thigh_pitch_joint
- removed joint right_shoulder_yaw_link
- added joint left_elbow_yaw_joint: type revolute, parent left_elbow_pitch_link, child left_elbow_yaw_link, origin xyz=0 0 -0.0133504827638016 rpy=0 0 0, axis 1 0 0, limit lower=-3.14159 upper=3.14159 effort=30 velocity=12
- added joint right_shoulder_yaw_joint: type revolute, parent right_shoulder_roll_link, child right_shoulder_yaw_link, origin xyz=0 -0.00647168056291525 0.000825647150946768 rpy=0 0 0, axis 0 0 -1, limit lower=-3.14159 upper=3.14159 effort=30 velocity=12
- added joint right_thigh_pitch_joint: type revolute, parent base_link, child right_thigh_pitch_link, origin xyz=0.043915 -0.1256 -0.036743 rpy=0 0 0, axis 0 -1 0, limit lower=-2.862 upper=2.862 effort=140 velocity=1.2
- joint right_thigh_roll_joint: parent right _thigh_pitch_link -> right_thigh_pitch_link
